Commit message: first commit

File: src/mybot/urdf/st.xacro (robot description, xacro)
@@ -2,54 +2,45 @@
 <robot name="st" xmlns:xacro="http://www.ros.org/wiki/xacro">
   <xacro:include filename="$(find mybot)/urdf/st.gazebo"/>
-  <link name='chassis'>
-    <pose>0 0 0.1 0 0 0</pose>
-    <inertial>
-      <mass value="5.0"/>
-      <origin xyz="0.0 0 0.1" rpy=" 0 0 0"/>
-      <inertia
-          ixx="0.1" ixy="0" ixz="0"
-          iyy="0.1" iyz="0"
-          izz="0.1"
-      />
-    </inertial>
-    <collision name='collision'>
-      <geometry>
-        <box size=".4 .2 .1"/>
-      </geometry>
-    </collision>
-    <visual name='chassis_visual'>
-      <origin xyz="0 0 0" rpy=" 0 0 0"/>
-      <geometry>
-        <box size=".4 .2 .1"/>
-      </geometry>
-        <material name="grey">
-    <color rgba="0.5 0.5 0.5 1.0"/>
-  </material>
-    </visual>
-    <visual name='chassis_visual_top'>
-      <origin xyz="-0.1 0 0.05" rpy=" 0 0 0"/>
-      <geometry>
-        <box size=".2 .1 .08"/>
-      </geometry>
-        <material name="green">
-    <color rgba="0.0 0.8 0.0 1.0"/>
-  </material>
-    </visual>
-    <collision name='caster_front_collision'>
-      <origin xyz="0.15 0 -0.05" rpy=" 0 0 0"/>
-      <geometry>
-        <sphere radius="0.05"/>
-      </geometry>
-    </collision>
-    <visual name='caster_front_visual'>
-      <origin xyz="0.15 0 -0.05" rpy=" 0 0 0"/>
-      <geometry>
-        <sphere radius="0.05"/>
-      </geometry>
-        <material name="black">
-    <color rgba="0.0 0.0 0.0 1.0"/>
-  </material>
-    </visual>
+  <link
+    name="base_link">
+    <inertial>
+      <origin
+        xyz="-0.037666 0.19446 0.026"
+        rpy="0 0 0" />
+      <mass
+        value="3" />
+      <inertia
+        ixx="0"
+        ixy="0"
+        ixz="0"
+        iyy="0"
+        iyz="0"
+        izz="0" />
+    </inertial>
+    <visual>
+      <origin
+        xyz="0 0 0"
+        rpy="0 0 0" />
+      <geometry>
+          <mesh
+            filename="package://mybot/meshes/container_link.STL" />
+      </geometry>
+      <material
+        name="">
+        <color
+          rgba="0.75294 0.75294 0.75294 1" />
+      </material>
+    </visual>
+    <collision>
+      <origin
+        xyz="0 0 0"
+        rpy="0 0 0" />
+      <geometry>
+          <mesh
+            filename="package://mybot/meshes/container_link.STL" />
+      </geometry>
+    </collision>
   </link>
+  <!--  Wheels -->
   <link name="left_wheel">
     <!--origin xyz="0.1 0.13 0.1" rpy="0 1.5707 1.5707"/-->
@@ -78,4 +69,12 @@
     </inertial>
   </link>
+  <joint type="continuous" name="left_wheel_hinge">
+    <origin xyz="-0.23 0.24887 0.033" rpy="0 0 0"/>
+    <child link="left_wheel"/>
+    <parent link="base_link"/>
+    <axis xyz="0 1 0" rpy="0 0 0"/>
+    <!-- <limit effort="10000" velocity="1000"/> -->
+    <joint_properties damping="2.0" friction="2.0"/>
+  </joint>
   <link name="right_wheel">
     <!--origin xyz="0.1 -0.13 0.1" rpy="0 1.5707 1.5707"/-->
@@ -104,47 +103,462 @@
     </inertial>
   </link>
-  <joint type="continuous" name="left_wheel_hinge">
-    <origin xyz="-0.1 0.15 0" rpy="0 0 0"/>
-    <!--origin xyz="0.1 0.13 0" rpy="0 1.5707 1.5707"/-->
-    <child link="left_wheel"/>
-    <parent link="chassis"/>
+  <joint type="continuous" name="right_wheel_hinge">
+    <origin xyz="-0.23 -0.24887 0.033" rpy="0 0 0"/>
+    <child link="right_wheel"/>
+    <parent link="base_link"/>
     <axis xyz="0 1 0" rpy="0 0 0"/>
     <!-- <limit effort="10000" velocity="1000"/> -->
-    <joint_properties damping="0.0" friction="0.0"/>
+    <joint_properties damping="2.0" friction="2.0"/>
   </joint>
-  <joint type="continuous" name="right_wheel_hinge">
-    <origin xyz="-0.1 -0.15 0" rpy="0 0 0"/>
-    <!--origin xyz="0.1 -0.13 0" rpy="0 1.5707 1.5707"/-->
-    <child link="right_wheel"/>
-    <parent link="chassis"/>
-    <axis xyz="0 1 0" rpy="0 0 0"/>
-    <!-- <limit effort="10000" velocity="1000"/> -->
-    <joint_properties damping="0.0" friction="0.0"/>
+<link name="wheel_front_left_link">
+    <inertial>
+      <origin
+        xyz="2.2922E-08 -3.5373E-10 0.00086907"
+        rpy="0 0 0" />
+      <mass
+        value="0.6" />
+      <inertia
+        ixx="0.00054477"
+        ixy="1.164E-11"
+        ixz="5.0249E-11"
+        iyy="0.00054477"
+        iyz="2.8527E-12"
+        izz="0.0010243" />
+    </inertial>
+    <visual>
+      <origin
+        xyz="0 0 0"
+        rpy="0 0 0" />
+      <geometry>
+        <cylinder radius="0.1" length="0.05"/>
+      </geometry>
+        <material name="black">
+            <color rgba="0.0 0.0 0.0 1.0"/>
+        </material>
+    </visual>
+    <collision>
+      <origin
+        xyz="0 0 0"
+        rpy="0 0 0" />
+      <geometry>
+        <cylinder radius="0.1" length="0.05"/>
+      </geometry>
+    </collision>
+</link>
+<joint name="joint_wheel_front_left"
+    type="continuous">
+    <origin
+      xyz="0.23 0.25887 0.033"
+      rpy="1.5708 0 3.1416" />
+    <parent
+      link="base_link" />
+    <child
+      link="wheel_front_left_link" />
+    <axis xyz="0 0 1" rpy="0 0 0"/>
+    <joint_properties damping="5.0" friction="5.0"/>
+</joint>
+<link name="wheel_front_right_link">
+    <inertial>
+      <origin
+        xyz="2.2203E-08 -5.7057E-09 0.00086907"
+        rpy="0 0 0" />
+      <mass
+        value="0.6" />
+      <inertia
+        ixx="0.00054477"
+        ixy="2.5356E-11"
+        ixz="4.9522E-11"
+        iyy="0.00054477"
+        iyz="-8.9807E-12"
+        izz="0.0010243" />
+    </inertial>
+    <visual>
+      <origin
+        xyz="0 0 0"
+        rpy="0 0 0" />
+      <geometry>
+        <cylinder radius="0.1" length="0.05"/>
+      </geometry>
+        <material name="black">
+            <color rgba="0.0 0.0 0.0 1.0"/>
+        </material>
+    </visual>
+    <collision>
+      <origin
+        xyz="0 0 0"
+        rpy="0 0 0" />
+      <geometry>
+        <cylinder radius="0.1" length="0.05"/>
+      </geometry>
+    </collision>
+</link>
+<joint name="joint_wheel_front_right"
+    type="continuous">
+    <origin
+      xyz="0.23 -0.25887 0.033"
+      rpy="1.5708 0 3.1416" />
+    <parent
+      link="base_link" />
+    <child
+      link="wheel_front_right_link" />
+    <axis xyz="0 0 1" rpy="0 0 0"/>
+    <joint_properties damping="5.0" friction="5.0"/>
+</joint>
+<transmission name="right_wheel_trans">
+  <type>transmission_interface/SimpleTransmission</type>
+  <actuator name="motor_right_wheel">
+    <hardwareInterface>EffortJointInterface</hardwareInterface>
+    <mechanicalReduction>1</mechanicalReduction>
+  </actuator>
+  <joint name="joint_wheel_front_right">
+    <hardwareInterface>VelocityJointInterface</hardwareInterface>
   </joint>
+</transmission>
+<transmission name="left_wheel_trans">
+  <type>transmission_interface/SimpleTransmission</type>
+  <actuator name="motor_left_wheel">
+    <hardwareInterface>EffortJointInterface</hardwareInterface>
+    <mechanicalReduction>1</mechanicalReduction>
+  </actuator>
+  <joint name="joint_wheel_front_left">
+    <hardwareInterface>VelocityJointInterface</hardwareInterface>
+  </joint>
+</transmission>
+<transmission name="right_wheel_hinge_trans">
+  <type>transmission_interface/SimpleTransmission</type>
+  <actuator name="motor_right_wheel_hinge">
+    <hardwareInterface>EffortJointInterface</hardwareInterface>
+    <mechanicalReduction>1</mechanicalReduction>
+  </actuator>
+  <joint name="right_wheel_hinge">
+    <hardwareInterface>VelocityJointInterface</hardwareInterface>
+  </joint>
+</transmission>
+<transmission name="left_wheel_hinge_trans">
+  <type>transmission_interface/SimpleTransmission</type>
+  <actuator name="motor_left_wheel_hinge">
+    <hardwareInterface>EffortJointInterface</hardwareInterface>
+    <mechanicalReduction>1</mechanicalReduction>
+  </actuator>
+  <joint name="left_wheel_hinge">
+    <hardwareInterface>VelocityJointInterface</hardwareInterface>
+  </joint>
+</transmission>
   <!-- Hokuyo Laser -->
-  <link name="hokuyo_link">
-    <collision>
-      <origin xyz="0 0 0" rpy="0 0 0"/>
-      <geometry>
-    <box size="0.1 0.1 0.1"/>
-      </geometry>
-    </collision>
-    <visual>
-      <origin xyz="0 0 0" rpy="0 0 0"/>
-      <geometry>
-        <mesh filename="package://mybot/meshes/hokuyo.dae"/>
-      </geometry>
-    </visual>
-    <inertial>
-      <mass value="1e-5" />
-      <origin xyz="0 0 0" rpy="0 0 0"/>
-      <inertia ixx="1e-6" ixy="0" ixz="0" iyy="1e-6" iyz="0" izz="1e-6" />
-    </inertial>
-  </link>
-  <joint name="hokuyo_joint" type="fixed">
+<link name="hokuyo_link">
+    <inertial>
+      <origin
+        xyz="-0.00064383 9.2927E-10 0.037832"
+        rpy="0 0 0" />
+      <mass
+        value="0.22916" />
+      <inertia
+        ixx="0.00020894"
+        ixy="1.295E-12"
+        ixz="-1.1307E-06"
+        iyy="0.00021335"
+        iyz="-4.2308E-12"
+        izz="0.00011244" />
+    </inertial>
+    <visual>
+      <origin
+        xyz="0 0 0"
+        rpy="0 0 0" />
+      <geometry>
+        <mesh
+          filename="package://mybot/meshes/lidar_point_link.STL" />
+      </geometry>
+      <material
+        name="">
+        <color
+          rgba="0 0 0 1" />
+      </material>
+    </visual>
+    <collision>
+      <origin
+        xyz="0 0 0"
+        rpy="0 0 0" />
+      <geometry>
+        <mesh
+          filename="package://mybot/meshes/lidar_point_link.STL" />
+      </geometry>
+    </collision>
+</link>
+<joint name="hokuyo_joint" type="fixed">
     <axis xyz="0 1 0" />
-    <origin xyz="0.15 0 0.1" rpy="0 0 0"/>
-    <parent link="chassis"/>
+    <origin
+      xyz="0.13 -0.0051 0.23"
+      rpy="0 0 0" />
+    <parent link="base_link"/>
     <child link="hokuyo_link"/>
-  </joint>
+</joint>
+ <!-- imu Link -->
+<link name="imu_sensor">
+    <visual>
+      <origin xyz="0.04 0 0.05" rpy="0 0 0"/>
+      <geometry>
+        <box size="0.07 0.07 0.03"/>
+      </geometry>
+      <material name="orange"/>
+    </visual>
+    <inertial>
+      <origin xyz="0 0 1" rpy="0 0 0"/>
+      <mass value="1"/>
+      <inertia
+        ixx="1.0" ixy="0.0" ixz="0.0"
+        iyy="1.0" iyz="0.0"
+        izz="1.0"/>
+    </inertial>
+</link>
+<joint name="sensor_joint" type="fixed">
+      <origin
+      xyz="0.1 0 0.0574"
+      rpy="0 0 0" />
+    <parent link="base_link"/>
+    <child link="imu_sensor"/>
+</joint>
+<!-- gps Link -->
+<link name="gps_link">
+    <inertial>
+      <origin
+        xyz="-0.002036 -0.001601 0.004"
+        rpy="0 0 0" />
+      <mass
+        value="0.0056708" />
+      <inertia
+        ixx="2.7399E-07"
+        ixy="8.0779E-24"
+        ixz="-1.5978E-22"
+        iyy="4.8412E-07"
+        iyz="-8.3674E-24"
+        izz="6.9802E-07" />
+    </inertial>
+    <visual>
+      <origin
+        xyz="0 0 0"
+        rpy="0 0 0" />
+      <geometry>
+        <mesh
+          filename="package://mybot/meshes/gps_ins_point_link.STL" />
+      </geometry>
+      <material
+        name="">
+        <color
+          rgba="1 0.50196 1 1" />
+      </material>
+    </visual>
+    <collision>
+      <origin
+        xyz="0 0 0"
+        rpy="0 0 0" />
+      <geometry>
+        <mesh
+          filename="package://mybot/meshes/gps_ins_point_link.STL" />
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